File: hardware/_autosave-kitchen-pcb.kicad_pcb (KiCad board)
At the start: 2 copper layers, 91.6 x 88 mm, 78 parts, among them IC1 ESP32-S3-WROOM-1-N8R8, J1 GSD090012SEU, J2 Conn_02x02_Odd_Even, J3 Conn_01x06, J4 Conn_01x03, J5 DCJ200-10-A-K1-K, J6 USB4105-GF-A, Q1 TEMT6000X01, SW1 SW_Push, SW2 SW_Push, U1 SHT30-DIS-B, U2 MX25L3233FM2I-08G, U3 NCP1117ST33T3G, U4 USBLC6-2SC6

Commit message: Layout v0.3
Parts:
- moved C15 72.6 mm to (112.5, 82.5), turned to 90 degrees
- moved R16 72.4 mm to (116.0, 82.5)
- moved H3 57.8 mm to (131.5, 95.5)
- moved R17 41.4 mm to (128.0, 61.0)
- moved D6 21.3 mm to (112.5, 92.5), turned to 0 degrees
- moved D8 19.3 mm to (109.0, 94.0), turned to -90 degrees
- moved R6 17.3 mm to (113.5, 95.5), turned to 90 degrees
- moved R15 16.6 mm to (161.3, 110.2), turned to -90 degrees
- moved R8 16.2 mm to (111.0, 96.0), turned to 90 degrees
- moved R14 14.6 mm to (173.0, 110.0), turned to -90 degrees
- moved Q1 12.5 mm to (161.3, 120.3)
- moved R10 12.5 mm to (160.3, 124.3)
- moved C11 11.7 mm to (163.8, 107.2), turned to 180 degrees
- moved TP2 11.7 mm to (135.9, 55.0)
- moved TP4 11.7 mm to (146.0, 55.0)
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Other:
- board size 91.6 x 88 mm -> 81.1 x 88.1 mm
