File: hardware/_autosave-untitled.kicad_sch (KiCad schematic)
At the start: 41 parts, among them J5 DCJ200-10-A-K1-K, J6 USB4105-GF-A, SW1 SW_Push, SW2 SW_Push, U3 NCP1117ST33T3G, U4 ESP32-S3-WROOM-1-N8R8, U5 USBLC6-2SC6

Commit message: Layout v0.6.2, SW1 footprint
Parts:
- SW1: renamed from S1; footprint R1966ABLKBLKGR -> ESP32-project-footprints:RA1113112R
- renumbered SW1 to SW2, SW2 to SW3
Other:
- note removed: "NEW SWITCH"
Changed lines of the file:
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@@
 		)
 	)
-	(text "NEW SWITCH	"
-		(exclude_from_sim no)
-		(at 168.656 22.606 0)
-		(effects
-			(font
-				(size 1.27 1.27)
-			)
-			(href "https://www.tme.eu/cz/details/ra1113112r/prepinace-rocker/e-switch/")
-		)
-	)
 	(text "NOTE: We are diode ORing between the\n2 power sources This means that if both\nUSB and DC jack are plugged in\nthe higer voltage will power the LDO"
 		(exclude_from_sim no)
@@
 		(dnp no)
 		(fields_autoplaced yes)
-		(property "Reference" "SW1"
+		(property "Reference" "SW2"
 			(at 36.83 73.66 0)
 			(effects
@@
 			(project "kitchen-pcb"
 				(path "/09f81662-95cc-469f-af04-c6a14137ce30/88485db4-61a5-4171-9283-b7e1247b6206"
-					(reference "SW1")
+					(reference "SW2")
 					(unit 1)
 				)
@@
 		(dnp no)
 		(fields_autoplaced yes)
-		(property "Reference" "SW2"
+		(property "Reference" "SW3"
 			(at 83.82 73.66 0)
 			(effects
@@
 			(project "kitchen-pcb"
 				(path "/09f81662-95cc-469f-af04-c6a14137ce30/88485db4-61a5-4171-9283-b7e1247b6206"
-					(reference "SW2")
+					(reference "SW3")
 					(unit 1)
 				)
@@
 		(on_board yes)
 		(dnp no)
-		(property "Reference" "S1"
+		(property "Reference" "SW1"
 			(at 169.672 26.924 90)
 			(effects
@@
 			)
 		)
-		(property "Footprint" "R1966ABLKBLKGR"
+		(property "Footprint" "ESP32-project-footprints:RA1113112R"
 			(at 258.75 22.86 0)
 			(effects
@@
 			(project ""
 				(path "/09f81662-95cc-469f-af04-c6a14137ce30/88485db4-61a5-4171-9283-b7e1247b6206"
-					(reference "S1")
+					(reference "SW1")
 					(unit 1)
 				)
